Commit message: almost there

File: UR5_ros/src/visualisation/urdf/gripper.urdf.xacro (robot description, xacro)
@@ -4,5 +4,5 @@
         <visual>
             <geometry>
-                <box size="0.1 0.1 0.02"/> <!-- Base dimensions adjusted -->
+                <box size="0.05 0.15 0.06"/> <!-- Base dimensions adjusted -->
             </geometry>
             <material name="gray">
@@ -12,10 +12,10 @@
     </link>
     <!-- Left finger -->
-    <link name="left_finger">
+    <link name="jaw_lead">
         <visual>
             <geometry>
-                <box size="0.02 0.02 0.1"/> <!-- Finger size -->
+                <box size="0.08 0.005 0.1"/> <!-- Finger size -->
             </geometry>
-            <origin xyz="0.0 0.05 0.0"/>
+            <origin xyz="-0.015 0.05 0.03"/>
             <material name="blue">
                 <color rgba="0.0 0.0 1.0 1"/>
@@ -24,16 +24,16 @@
         <collision>
             <geometry>
-                <box size="0.02 0.02 0.1"/> <!-- Collision geometry matches visual -->
+                <box size="0.08 0.005 0.1"/> <!-- Collision geometry matches visual -->
             </geometry>
-            <origin xyz="0.0 0.05 0.0"/>
+            <origin xyz="-0.015 0.05 0.03"/>
         </collision>
     </link>
     <!-- Right finger -->
-    <link name="right_finger">
+    <link name="jaw_follow">
         <visual>
             <geometry>
-                <box size="0.02 0.02 0.1"/> <!-- Finger size -->
+                <box size="0.08 0.005 0.1"/> <!-- Finger size -->
             </geometry>
-            <origin xyz="0.0 -0.05 0.0"/>
+            <origin xyz="-0.015 -0.05 0.03"/>
             <material name="red">
                 <color rgba="1.0 0.0 0.0 1"/>
@@ -42,24 +42,25 @@
         <collision>
             <geometry>
-                <box size="0.02 0.02 0.1"/> <!-- Collision geometry matches visual -->
+                <box size="0.08 0.005 0.1"/> <!-- Collision geometry matches visual -->
             </geometry>
-            <origin xyz="0.0 -0.05 0.0"/>
+            <origin xyz="-0.015 -0.05 0.03"/>
         </collision>
     </link>
     <!-- Left finger joint (prismatic for symmetric opening) -->
-    <joint name="left_joint" type="prismatic">
+    <joint name="main_joint" type="prismatic">
         <parent link="base_link"/>
-        <child link="left_finger"/>
-        <origin xyz="0.0 0.05 0.0" rpy="0 0 0"/>
-        <axis xyz="0 1 0"/>
+        <child link="jaw_lead"/>
+        <origin xyz="0.0 0.0 0.0" rpy="0 0 0"/>
+        <axis xyz="0 -1 0"/>
         <limit lower="0" upper="0.05" effort="1.0" velocity="0.5"/>
     </joint>
     <!-- Right finger joint (prismatic for symmetric opening) -->
-    <joint name="right_joint" type="prismatic">
+    <joint name="follow_joint" type="prismatic">
         <parent link="base_link"/>
-        <child link="right_finger"/>
-        <origin xyz="0.0 -0.05 0.0" rpy="0 0 0"/>
-        <axis xyz="0 -1 0"/>
+        <child link="jaw_follow"/>
+        <origin xyz="0.0 0.0 0.0" rpy="0 0 0"/>
+        <axis xyz="0 1 0"/>
         <limit lower="0" upper="0.05" effort="1.0" velocity="0.5"/>
+        <mimic joint="main_joint" multiplyer="1.0"/>
     </joint>
 </robot>

Commit message: moar

File: UR5_ros/src/visualisation/urdf/gripper.urdf.xacro (robot description, xacro)
@@ -1,5 +1,5 @@
 <robot name="gripper" xmlns:xacro="http://ros.org/wiki/xacro">
     <!-- Base link -->
-    <link name="base_link">
+    <link name="link_0">
         <visual>
             <geometry>
@@ -10,4 +10,9 @@
             </material>
         </visual>
+        <collision>
+            <geometry>
+                <box size="0.05 0.15 0.06"/> <!-- Collision geometry matches visual -->
+            </geometry>
+        </collision>
     </link>
     <!-- Left finger -->
@@ -49,5 +54,5 @@
     <!-- Left finger joint (prismatic for symmetric opening) -->
     <joint name="main_joint" type="prismatic">
-        <parent link="base_link"/>
+        <parent link="link_0"/>
         <child link="jaw_lead"/>
         <origin xyz="0.0 0.0 0.0" rpy="0 0 0"/>
@@ -57,5 +62,5 @@
     <!-- Right finger joint (prismatic for symmetric opening) -->
     <joint name="follow_joint" type="prismatic">
-        <parent link="base_link"/>
+        <parent link="link_0"/>
         <child link="jaw_follow"/>
         <origin xyz="0.0 0.0 0.0" rpy="0 0 0"/>

Commit message: bit of a mess but main fule being worked on is ur5_grip_launch, adapted from a forum post, it was working but now it gives me a segfault

File: UR5_ros/src/visualisation/urdf/gripper.urdf.xacro (robot description, xacro)
@@ -1,5 +1,21 @@
+<!-- <?xml version="1.0"?> -->
 <robot name="gripper" xmlns:xacro="http://ros.org/wiki/xacro">
     <!-- Base link -->
     <link name="gripper_base">
+        <visual>
+            <geometry>
+                <cylinder radius="0.025" length="0.07"/> <!-- Base dimensions adjusted -->
+            </geometry>
+            <material name="gray">
+                <color rgba="0.5 0.5 0.5 1"/>
+            </material>
+        </visual>
+        <collision>
+            <geometry>
+                <cylinder radius="0.025" length="0.07"/> <!-- Collision geometry matches visual -->
+            </geometry>
+        </collision>
+    </link>
+    <link name="slider">
         <visual>
             <geometry>
@@ -52,7 +68,12 @@
         </collision>
     </link>
+    <joint name = "base_joint" type = "fixed">
+        <parent link = "gripper_base"/>
+        <child link = "slider"/>
+        <origin xyz="0.0 0.0 0.0" rpy="0 0 0"/>
+    </joint>
     <!-- Left finger joint (prismatic for symmetric opening) -->
-    <joint name="main_joint" type="prismatic">
-        <parent link="gripper_base"/>
+    <joint name="right_finger_joint" type="prismatic">
+        <parent link="slider"/>
         <child link="jaw_lead"/>
         <origin xyz="0.0 0.0 0.0" rpy="0 0 0"/>
@@ -61,11 +82,11 @@
     </joint>
     <!-- Right finger joint (prismatic for symmetric opening) -->
-    <joint name="follow_joint" type="prismatic">
-        <parent link="gripper_base"/>
+    <joint name="left_finger_joint" type="prismatic">
+        <mimic joint="right_finger_joint" multiplyer="1.0"/>
+        <parent link="slider"/>
         <child link="jaw_follow"/>
         <origin xyz="0.0 0.0 0.0" rpy="0 0 0"/>
         <axis xyz="0 1 0"/>
         <limit lower="0" upper="0.05" effort="1.0" velocity="0.5"/>
-        <mimic joint="main_joint" multiplyer="1.0"/>
     </joint>
 </robot>

File: UR5_ros/src/visualisation/urdf/ur5_with_gripper.urdf.xacro (robot description, xacro)
@@ -1,3 +1,4 @@
-<robot name="ur_with_gripper" xmlns:xacro="http://www.ros.org/wiki/xacro" >
+<!-- <?xml version="1.0"?> -->
+<robot name="ur5_with_gripper" xmlns:xacro="http://www.ros.org/wiki/xacro" >
   <!-- UR5e robot arm -->
   <!-- URDF won't build if following args aren't defined. -->
@@ -6,5 +7,5 @@
   <xacro:include filename="$(find ur_description)/urdf/ur.urdf.xacro"/>
   <!-- end effector -->
-  <xacro:include filename="$(find visualisation)/urdf/gripper.xacro" />
+  <xacro:include filename="$(find visualisation)/urdf/gripper.urdf.xacro" />
   <!-- Coupler between arm and end effector -->
   <joint name="ur5_gripper_coupler_joint" type="fixed">
