Commit message: setting up rviz

File: UR5_ros/src/visualisation/urdf/gripper.xacro (robot description, xacro)
@@ -1,5 +1,5 @@
 <robot name="gripper" xmlns:xacro="http://ros.org/wiki/xacro">
     <!-- Base link -->
-    <link name="link_0">
+    <link name="gripper_base">
         <visual>
             <geometry>
@@ -54,5 +54,5 @@
     <!-- Left finger joint (prismatic for symmetric opening) -->
     <joint name="main_joint" type="prismatic">
-        <parent link="link_0"/>
+        <parent link="gripper_base"/>
         <child link="jaw_lead"/>
         <origin xyz="0.0 0.0 0.0" rpy="0 0 0"/>
@@ -62,5 +62,5 @@
     <!-- Right finger joint (prismatic for symmetric opening) -->
     <joint name="follow_joint" type="prismatic">
-        <parent link="link_0"/>
+        <parent link="gripper_base"/>
         <child link="jaw_follow"/>
         <origin xyz="0.0 0.0 0.0" rpy="0 0 0"/>

File: UR5_ros/src/visualisation/urdf/ur5_with_gripper.xacro (robot description, xacro)
@@ -1,3 +1,2 @@
-<?xml version="1.0" ?>
 <robot name="ur_with_gripper" xmlns:xacro="http://www.ros.org/wiki/xacro" >
   <!-- UR5e robot arm -->
@@ -9,5 +8,5 @@
   <xacro:include filename="$(find visualistion)/urdf/gripper.urdf.xacro" />
   <!-- Coupler between arm and end effector -->
-  <joint name="ur5_pizza_gripper_coupler_joint" type="fixed">
+  <joint name="ur5_gripper_coupler_joint" type="fixed">
     <parent link="tool0"/>
     <child link="link_0"/>

Commit message: robot description now publishes properly, but gripper joints are not dynamic

File: UR5_ros/src/visualisation/urdf/gripper.xacro (robot description, xacro)
@@ -5,5 +5,5 @@
         <visual>
             <geometry>
-                <cylinder radius="0.025" length="0.07"/> <!-- Base dimensions adjusted -->
+                <cylinder radius="0.025" length="0.03"/> <!-- Base dimensions adjusted -->
             </geometry>
             <material name="gray">
@@ -20,5 +20,5 @@
         <visual>
             <geometry>
-                <box size="0.05 0.15 0.06"/> <!-- Base dimensions adjusted -->
+                <box size="0.05 0.15 0.05"/> <!-- Base dimensions adjusted -->
             </geometry>
             <material name="gray">
@@ -36,7 +36,6 @@
         <visual>
             <geometry>
-                <box size="0.08 0.005 0.1"/> <!-- Finger size -->
+                <box size="0.08 0.005 0.05"/> <!-- Finger size -->
             </geometry>
-            <origin xyz="-0.015 0.05 0.03"/>
             <material name="blue">
                 <color rgba="0.0 0.0 1.0 1"/>
@@ -45,7 +44,6 @@
         <collision>
             <geometry>
-                <box size="0.08 0.005 0.1"/> <!-- Collision geometry matches visual -->
+                <box size="0.08 0.005 0.05"/> <!-- Collision geometry matches visual -->
             </geometry>
-            <origin xyz="-0.015 0.05 0.03"/>
         </collision>
     </link>
@@ -54,7 +52,6 @@
         <visual>
             <geometry>
-                <box size="0.08 0.005 0.1"/> <!-- Finger size -->
+                <box size="0.08 0.005 0.05"/> <!-- Finger size -->
             </geometry>
-            <origin xyz="-0.015 -0.05 0.03"/>
             <material name="red">
                 <color rgba="1.0 0.0 0.0 1"/>
@@ -63,30 +60,29 @@
         <collision>
             <geometry>
-                <box size="0.08 0.005 0.1"/> <!-- Collision geometry matches visual -->
+                <box size="0.08 0.005 0.05"/> <!-- Collision geometry matches visual -->
             </geometry>
-            <origin xyz="-0.015 -0.05 0.03"/>
         </collision>
     </link>
-    <joint name = "base_joint" type = "fixed">
+    <joint name = "gripper_base_joint" type = "fixed">
         <parent link = "gripper_base"/>
         <child link = "slider"/>
-        <origin xyz="0.0 0.0 0.0" rpy="0 0 0"/>
+        <origin xyz="0.0 0.0 0.04" rpy="0 0 0"/>
     </joint>
     <!-- Left finger joint (prismatic for symmetric opening) -->
-    <joint name="right_finger_joint" type="prismatic">
+    <joint name="right_finger_joint" type="fixed">
         <parent link="slider"/>
         <child link="jaw_lead"/>
-        <origin xyz="0.0 0.0 0.0" rpy="0 0 0"/>
+        <origin xyz="-0.015 0.05 0.055" rpy="0 0 0"/>
         <axis xyz="0 -1 0"/>
-        <limit lower="0" upper="0.05" effort="1.0" velocity="0.5"/>
+        <!-- <limit lower="0" upper="0.05" effort="1.0" velocity="0.5"/> -->
     </joint>
     <!-- Right finger joint (prismatic for symmetric opening) -->
-    <joint name="left_finger_joint" type="prismatic">
+    <joint name="left_finger_joint" type="fixed">
         <mimic joint="right_finger_joint" multiplyer="1.0"/>
         <parent link="slider"/>
         <child link="jaw_follow"/>
-        <origin xyz="0.0 0.0 0.0" rpy="0 0 0"/>
+        <origin xyz="-0.015 -0.05 0.055" rpy="0 0 0"/>
         <axis xyz="0 1 0"/>
-        <limit lower="0" upper="0.05" effort="1.0" velocity="0.5"/>
+        <!-- <limit lower="0" upper="0.05" effort="1.0" velocity="0.5"/> -->
     </joint>
 </robot>

File: UR5_ros/src/visualisation/urdf/ur5_with_gripper.xacro (robot description, xacro)
@@ -7,5 +7,5 @@
   <xacro:include filename="$(find ur_description)/urdf/ur.urdf.xacro"/>
   <!-- end effector -->
-  <xacro:include filename="$(find visualisation)/urdf/gripper.urdf.xacro" />
+  <xacro:include filename="$(find visualisation)/urdf/gripper.xacro" />
   <!-- Coupler between arm and end effector -->
   <joint name="ur5_gripper_coupler_joint" type="fixed">

Commit message: fixed collision

File: UR5_ros/src/visualisation/urdf/gripper.xacro (robot description, xacro)
@@ -11,9 +11,9 @@
             </material>
         </visual>
-        <collision>
+        <!-- <collision>
             <geometry>
-                <cylinder radius="0.025" length="0.07"/> <!-- Collision geometry matches visual -->
+                <cylinder radius="0.025" length="0.07"/>
             </geometry>
-        </collision>
+        </collision> -->
     </link>
     <link name="slider">
@@ -23,10 +23,10 @@
             </geometry>
             <material name="gray">
-                <color rgba="0.5 0.5 0.5 1"/>
+                <color rgba="0.3 0.3 0.3 1"/>
             </material>
         </visual>
         <collision>
             <geometry>
-                <box size="0.05 0.15 0.06"/> <!-- Collision geometry matches visual -->
+                <box size="0.05 0.15 0.05"/> <!-- Collision geometry matches visual -->
             </geometry>
         </collision>
@@ -39,10 +39,10 @@
             </geometry>
             <material name="blue">
-                <color rgba="0.0 0.0 1.0 1"/>
+                <color rgba="0.0 0.3 1.0 1"/>
             </material>
         </visual>
         <collision>
             <geometry>
-                <box size="0.08 0.005 0.05"/> <!-- Collision geometry matches visual -->
+                <box size="0.08 0.005 0.03"/>
             </geometry>
         </collision>
@@ -54,12 +54,13 @@
                 <box size="0.08 0.005 0.05"/> <!-- Finger size -->
             </geometry>
-            <material name="red">
-                <color rgba="1.0 0.0 0.0 1"/>
+            <material name="blue">
+                <color rgba="0.0 0.3 1.0 1"/>
             </material>
         </visual>
         <collision>
             <geometry>
-                <box size="0.08 0.005 0.05"/> <!-- Collision geometry matches visual -->
+                <box size="0.08 0.005 0.03"/>
             </geometry>
+            <origin xyz="0.0 0.0 0.01" rpy="0.0 0.0 0.0"/>
         </collision>
     </link>

File: UR5_ros/src/visualisation/urdf/ur5_with_gripper.xacro (robot description, xacro)
@@ -12,4 +12,5 @@
     <parent link="tool0"/>
     <child link="gripper_base"/>
+    <origin xyz="0.0 0.0 0.0" rpy="0.0 0.0 0.0"/>
   </joint>
 </robot>
